File: src/uru-card.brd (EAGLE design)
At the start: 54 x 85.6 mm, 46 parts, among them U1 ESP32-PICO-D4, U2 MPR121QR2, U3 AP2112K-3.3TRG1, U4 FT260Q-T, U6 ATECC508A-UDFN

Commit message: Updated CAM job
Parts:
- renumbered U$1 to J1, U$10 to TP9, U$11 to TP10, U$12 to TP11, U$13 to TP12, U$14 to D1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
